Commit message: change link name and add usd

File: robots/mevius/mevius.urdf (robot description, URDF)
Before this commit: robot mevius, 17 links, 16 joints
Links:
- removed link BL_calf_link
- removed link BL_foot_link
- removed link BL_scapula_link
- removed link BL_thigh_link
- removed link BR_calf_link
- removed link BR_foot_link
- removed link BR_scapula_link
- removed link BR_thigh_link
- removed link FL_calf_link
- removed link FL_foot_link
- removed link FL_scapula_link
- removed link FL_thigh_link
- removed link FR_calf_link
- removed link FR_foot_link
- removed link FR_scapula_link
- removed link FR_thigh_link
- removed link base_link
- added link BL_calf, mass 0.101512760080133; collision cylinder length=0.23 radius=0.01; visual mesh filename=meshes/BL_calf.STL
- added link BL_foot, mass 0.05; collision sphere radius=0.025; visual sphere radius=0.025
- added link BL_scapula, mass 0.792389082205849; collision cylinder length=0.08 radius=0.05; visual mesh filename=meshes/BL_scapula.STL
- added link BL_thigh, mass 1.28036049228712; visual mesh filename=meshes/BL_thigh.STL
- added link BR_calf, mass 0.101512760080133; collision cylinder length=0.23 radius=0.01; visual mesh filename=meshes/BR_calf.STL
- added link BR_foot, mass 0.05; collision sphere radius=0.025; visual sphere radius=0.025
- added link BR_scapula, mass 0.79239; collision cylinder length=0.08 radius=0.05; visual mesh filename=meshes/BR_scapula.STL
- added link BR_thigh, mass 1.28036049228712; visual mesh filename=meshes/BR_thigh.STL
- added link FL_calf, mass 0.101512760080133; collision cylinder length=0.23 radius=0.01; visual mesh filename=meshes/FL_calf.STL
- added link FL_foot, mass 0.05; collision sphere radius=0.025; visual sphere radius=0.025
- added link FL_scapula, mass 0.79238908220585; collision cylinder length=0.08 radius=0.05; visual mesh filename=meshes/FL_scapula.STL
- added link FL_thigh, mass 1.28036049228712; visual mesh filename=meshes/FL_thigh.STL
- added link FR_calf, mass 0.101512760080133; collision cylinder length=0.23 radius=0.01; visual mesh filename=meshes/FR_calf.STL
- added link FR_foot, mass 0.05; collision sphere radius=0.025; visual sphere radius=0.025
- added link FR_scapula, mass 0.79238908220585; collision cylinder length=0.08 radius=0.05; visual mesh filename=meshes/FR_scapula.STL
- added link FR_thigh, mass 1.28036049228712; visual mesh filename=meshes/FR_thigh.STL
- added link base, mass 8.0; collision box size=0.334 0.200 0.150; visual mesh filename=meshes/base.STL
Joints:
- removed joint BL_collar
- removed joint BL_hip
- removed joint BL_knee
- removed joint BR_collar
- removed joint BR_hip
- removed joint BR_knee
- removed joint FL_collar
- removed joint FL_hip
- removed joint FL_knee
- removed joint FR_collar
- removed joint FR_hip
- removed joint FR_knee
- added joint BL_collar_joint: type revolute, parent base, child BL_scapula, origin xyz=-0.16405000000001 0.0719999999999999 0.0564999653300497 rpy=0 0 0, axis 1 0 0, limit lower=-0.7854 upper=0.7854 effort=25 velocity=310
- added joint BL_hip_joint: type revolute, parent BL_scapula, child BL_thigh, origin xyz=-0.0555000000000055 0.01205000000001 0 rpy=0 0 0, axis 0 1 0, limit lower=0.0 upper=1.5708 effort=25 velocity=310
- added joint BL_knee_joint: type revolute, parent BL_thigh, child BL_calf, origin xyz=0 0.06555 -0.25 rpy=0 0 0, axis 0 1 0, limit lower=-2.8745 upper=-1.08 effort=25 velocity=310
- added joint BR_collar_joint: type revolute, parent base, child BR_scapula, origin xyz=-0.16405000000001 -0.0719999999999995 0.0565000000000019 rpy=0 0 0, axis 1 0 0, limit lower=-0.7854 upper=0.7854 effort=25 velocity=310
- added joint BR_hip_joint: type revolute, parent BR_scapula, child BR_thigh, origin xyz=-0.0555000000000055 -0.01205000000001 0 rpy=0 0 0, axis 0 1 0, limit lower=0.0 upper=1.5708 effort=25 velocity=310
- added joint BR_knee_joint: type revolute, parent BR_thigh, child BR_calf, origin xyz=0 -0.06555 -0.25 rpy=0 0 0, axis 0 1 0, limit lower=-2.8745 upper=-1.08 effort=25 velocity=310
- added joint FL_collar_joint: type revolute, parent base, child FL_scapula, origin xyz=0.16405000000001 0.0720000000000002 0.056500000000002 rpy=0 0 0, axis 1 0 0, limit lower=-0.7854 upper=0.7854 effort=25 velocity=310
- added joint FL_hip_joint: type revolute, parent FL_scapula, child FL_thigh, origin xyz=0.0555000000000021 0.01205000000001 0 rpy=0 0 0, axis 0 1 0, limit lower=0.0 upper=1.5708 effort=25 velocity=310
- added joint FL_knee_joint: type revolute, parent FL_thigh, child FL_calf, origin xyz=0 0.06555000000001 -0.250000000000004 rpy=0 0 0, axis 0 1 0, limit lower=-2.8745 upper=-1.08 effort=25 velocity=310
- added joint FR_collar_joint: type revolute, parent base, child FR_scapula, origin xyz=0.16405000000001 -0.0720000000000002 0.056500000000002 rpy=0 0 0, axis 1 0 0, limit lower=-0.7854 upper=0.7854 effort=25 velocity=310
- added joint FR_hip_joint: type revolute, parent FR_scapula, child FR_thigh, origin xyz=0.0555000000000021 -0.01205000000001 0 rpy=0 0 0, axis 0 1 0, limit lower=0.0 upper=1.5708 effort=25 velocity=310
- added joint FR_knee_joint: type revolute, parent FR_thigh, child FR_calf, origin xyz=0 -0.06555000000001 -0.250000000000004 rpy=0 0 0, axis 0 1 0, limit lower=-2.8745 upper=-1.08 effort=25 velocity=310
- joint BL_ankle_joint: child BL_foot_link -> BL_foot; parent BL_calf_link -> BL_calf
- joint BR_ankle_joint: child BR_foot_link -> BR_foot; parent BR_calf_link -> BR_calf
- joint FL_ankle_joint: child FL_foot_link -> FL_foot; parent FL_calf_link -> FL_calf
- joint FR_ankle_joint: child FR_foot_link -> FR_foot; parent FR_calf_link -> FR_calf
